Commit message: correctly implemented the PID controller, added the apply_wrench node

File: urdf/robot.urdf (robot description, URDF)
Before this commit: robot robot, 8 links, 7 joints
Joints:
- joint arm_height_joint: axis (none) -> 0 0 1; limit lower=-0.6 upper=0 effort=10 velocity=0.5 -> lower=-0.6 upper=0 effort=5000 velocity=0.5
- joint arm_rotation_joint: limit lower=-1.5708 upper=0 effort=10 velocity=0.5 -> lower=-1.5708 upper=0 effort=5000 velocity=0.5
- joint base_rotation_joint: limit lower=-3.141 upper=1.5708 effort=1000 velocity=0.5 -> lower=-3.141 upper=1.5708 effort=5000 velocity=0.5

Commit message: Fix: URDF arm_rotation_joint upper limit from 0 to -pi

File: urdf/robot.urdf (robot description, URDF)
Before this commit: robot robot, 8 links, 7 joints
Joints:
- joint arm_rotation_joint: limit lower=-1.5708 upper=0 effort=5000 velocity=0.5 -> lower=-1.5708 upper=-3.141 effort=5000 velocity=0.5

Commit message: Fix: URDF arm_rotation_joint lower limit from -pi/2 to 0

File: urdf/robot.urdf (robot description, URDF)
Before this commit: robot robot, 8 links, 7 joints
Joints:
- joint arm_rotation_joint: limit lower=-1.5708 upper=-3.141 effort=5000 velocity=0.5 -> lower=0 upper=-3.141 effort=5000 velocity=0.5

Commit message: :Feat: somewhat OK reference trajectory

File: urdf/robot.urdf (robot description, URDF)
Before this commit: robot robot, 8 links, 7 joints
Joints:
- joint arm_rotation_joint: limit lower=0 upper=-3.141 effort=5000 velocity=0.5 -> lower=-3.141 upper=0 effort=5000 velocity=0.5

Commit message: Updated Robot Base and First Motor block

File: urdf/robot.urdf (robot description, URDF)
Before this commit: robot robot, 8 links, 7 joints
Links:
- removed link arm_connection
- removed link arm_first_link
- removed link arm_second_link
- removed link arm_third_link
- removed link base_cylinder
- removed link bed_and_base
- removed link end_effector
- added link base_cube_link, mass 10; collision box size=0.218 0.2165 0.210; visual box size=0.218 0.2165 0.210
- added link robot_base_link, mass 10; collision box size=0.395 0.555 0.08; visual box size=0.395 0.555 0.08
Joints:
- removed joint arm_first_joint
- removed joint arm_height_joint
- removed joint arm_rotation_joint
- removed joint arm_second_joint
- removed joint base_rotation_joint
- removed joint end_effector_joint
- added joint base_cube_cylinder_joint: type fixed, parent base_cube_link, child telescope_outside_link, origin xyz=0 0 0.08
- added joint robot_base_base_cube_joint: type fixed, parent robot_base_link, child base_cube_link, origin xyz=0 0 0.08
- joint map_robot_joint: child bed_and_base -> robot_base_link

Commit message: remodelling robot by hand

File: urdf/robot.urdf (robot description, URDF)
Before this commit: robot robot, 3 links, 3 joints
Links:
- removed link base_cube_link
- removed link map
- removed link robot_base_link
- added link column_inside_link, mass 10.0; collision box size=0.120 0.177 0.640; visual box size=0.120 0.177 0.640
- added link column_outside_link, mass 10.0; collision box size=0.010 0.202 0.640; visual box size=0.010 0.202 0.640
- added link frame_link, mass 100.0; collision box size=1.395 0.645 0.080; visual box size=1.395 0.645 0.080
- added link lower_motor_box_link, mass 10.0; collision box size=0.2165 0.218 0.220; visual box size=0.2165 0.218 0.220
- added link middle_motor_box_link, mass 10.0; collision box size=0.218 0.218 0.170; visual box size=0.218 0.218 0.170
- added link robot_base
- added link upper_cylinder_link, mass 10.0; collision cylinder length=0.040 radius=0.110; visual cylinder length=0.040 radius=0.110
- added link upper_motor_box_link, mass 10.0; collision box size=0.4215 0.223 0.1695; visual box size=0.4215 0.223 0.1695
Joints:
- removed joint base_cube_cylinder_joint
- removed joint map_robot_joint
- removed joint robot_base_base_cube_joint
- added joint column_inside_joint: type fixed, parent column_inside_link, child middle_motor_box_link, origin xyz=0 0 0.650
- added joint column_outside_column_inside_joint: type prismatic, parent column_outside_link, child column_inside_link, origin xyz=0 0 0.005, axis 0 0 1, limit lower=0.005 upper=0.165 effort=5000 velocity=0.5
- added joint frame_lower_motor_box_joint: type fixed, parent frame_link, child lower_motor_box_link, origin xyz=-0.35575 0.180 0.080
- added joint lower_motor_box_column_outside_joint: type fixed, parent lower_motor_box_link, child column_outside_link, origin xyz=0 0 0.220
- added joint map_frame_joint: type fixed, parent robot_base, child frame_link, origin xyz=0.35575 -0.180 0
- added joint middle_box_upper_cylinder_joint: type fixed, parent middle_motor_box_link, child upper_cylinder_link, origin xyz=0 0 0.170
- added joint upper_cylinder_upper_motor_joint: type revolute, parent upper_cylinder_link, child upper_motor_box_link, origin xyz=0 0 0.020, axis 0 0 1, limit lower=-3.141 upper=1.5708 effort=5000 velocity=0.5

Commit message: make controller compatible with new joints

File: urdf/robot.urdf (robot description, URDF)
Before this commit: robot robot, 8 links, 7 joints
Links:
- added link arm_first_link, mass 0.5; collision cylinder length=0.125742 radius=0.015; visual cylinder length=0.125742 radius=0.015
- added link arm_second_link, mass 1.1; collision cylinder length=0.300 radius=0.015; visual cylinder length=0.300 radius=0.015
- added link arm_third_link, mass 2.4; collision cylinder length=0.810 radius=0.015; visual cylinder length=0.810 radius=0.015
Joints:
- added joint arm_first_joint: type fixed, parent arm_first_link, child arm_second_link, origin xyz=0 0 0.161204 rpy=0 -1.5708 0
- added joint arm_second_joint: type fixed, parent arm_second_link, child arm_third_link, origin xyz=0.04 0 0.3 rpy=0 1.5708 0
- added joint upper_motor_box_arm_joint: type revolute, parent upper_motor_box_link, child arm_first_link, origin xyz=0.095 0 0.08475 rpy=0 -1.57079 3.1415926, axis 0 0 1, limit lower=-1.5708 upper=0 effort=5000 velocity=0.5

Commit message: adjusted mass

File: urdf/robot.urdf (robot description, URDF)
Before this commit: robot robot, 11 links, 10 joints
Links:
- added link end_effector
- link arm_first_link: mass 0.5 -> 1.5
- link arm_second_link: mass 1.1 -> 0.5
- link arm_third_link: mass 2.4 -> 2.5
- link column_inside_link: mass 10.0 -> 9.0
- link column_outside_link: mass 10.0 -> 9.0
- link lower_motor_box_link: mass 10.0 -> 19.5
- link middle_motor_box_link: mass 10.0 -> 19.0
- link upper_cylinder_link: mass 10.0 -> 1.0
- link upper_motor_box_link: mass 10.0 -> 22.0
Joints:
- removed joint column_outside_column_inside_joint
- removed joint upper_cylinder_upper_motor_joint
- removed joint upper_motor_box_arm_joint
- added joint arm_height_joint: type prismatic, parent column_outside_link, child column_inside_link, origin xyz=0 0 0.005, axis 0 0 1, limit lower=0.005 upper=0.165 effort=5000 velocity=0.5
- added joint arm_rotation_joint: type revolute, parent upper_motor_box_link, child arm_first_link, origin xyz=0.095 0 0.08475 rpy=0 -1.57079 3.1415926, axis 0 0 1, limit lower=-1.5708 upper=0 effort=5000 velocity=0.5
- added joint base_rotation_joint: type revolute, parent upper_cylinder_link, child upper_motor_box_link, origin xyz=0 0 0.020, axis 0 0 1, limit lower=-3.141 upper=1.5708 effort=5000 velocity=0.5
- added joint end_effector_joint: type fixed, parent arm_third_link, child end_effector, origin xyz=0 0 0 rpy=0 -1.5708 0

Commit message: updated arm geometry, added colors and calculated inertia properties

File: urdf/robot.urdf (robot description, URDF)
Before this commit: robot robot, 12 links, 11 joints
Links:
- link arm_first_link: geometry collision cylinder length=0.148 radius=0.015; visual cylinder length=0.148 radius=0.015
- link arm_second_link: geometry collision cylinder length=0.306 radius=0.015; visual cylinder length=0.306 radius=0.015
- link arm_third_link: geometry collision cylinder length=0.838 radius=0.015; visual cylinder length=0.838 radius=0.015
Joints:
- joint arm_first_joint: origin xyz=0 0 0.161204 rpy=0 -1.5708 0 -> xyz=0 0 0.148 rpy=0 -1.5708 0
- joint arm_second_joint: origin xyz=0.04 0 0.3 rpy=0 1.5708 0 -> xyz=0 0 0.314 rpy=0 1.5708 0
- joint base_rotation_joint: origin xyz=0 0 0.020 -> xyz=0 0 0.040

Commit message: adjusted joint names, corrected joint limits and types, correct yaml typo

File: urdf/robot.urdf (robot description, URDF)
Before this commit: robot robot, 12 links, 11 joints
Joints:
- removed joint arm_height_joint
- removed joint arm_rotation_joint
- removed joint base_rotation_joint
- added joint column_outside_column_inside_joint: type prismatic, parent column_outside_link, child column_inside_link, origin xyz=0 0 0.005, axis 0 0 1, limit lower=0 upper=50.0 effort=5000 velocity=100
- added joint upper_cylinder_upper_motor_joint: type continuous, parent upper_cylinder_link, child upper_motor_box_link, origin xyz=0 0 0.040, axis 0 0 1
- added joint upper_motor_box_arm_joint: type continuous, parent upper_motor_box_link, child arm_first_link, origin xyz=0.095 0 0.08475 rpy=0 -1.57079 3.1415926, axis 0 0 1
- joint end_effector_joint: origin xyz=0 0 0 rpy=0 -1.5708 0 -> xyz=0 0 0.2 rpy=0 -1.5708 0

Commit message: modified added bed, improved launch and pid controller file

File: urdf/robot.urdf (robot description, URDF)
Before this commit: robot robot, 12 links, 11 joints
Links:
- added link Bed_center_link, mass 2.0; collision box size=0.900 2.004 0.170; visual box size=0.900 2.004 0.170
- added link BodyArms_link, mass 9.0; collision box size=0.400 0.200 0.040; visual box size=0.400 0.200 0.040
- added link UpperBody_link, mass 9.0; collision box size=0.400 0.100 0.550; visual box size=0.400 0.100 0.550
- link column_outside_link: mass 9.0 -> 0.5
- link lower_motor_box_link: mass 19.5 -> 28.0
Joints:
- added joint BodyArms_UpperBody_joint: type fixed, parent BodyArms_link, child UpperBody_link, origin xyz=0 0.200 -0.100
- added joint column_outside_Bedcenter_joint: type fixed, parent column_outside_link, child Bed_center_link, origin xyz=0.774 0 0.120
- added joint robot_Body_joint: type continuous, parent arm_third_link, child BodyArms_link, origin xyz=0.015 0 0.419 rpy=0 1.5708 0, axis 1 0 0
- joint end_effector_joint: origin xyz=0 0 0.2 rpy=0 -1.5708 0 -> xyz=0 0 0.838 rpy=0 -1.5708 0

Commit message: advanced Body Links and joints

File: urdf/robot.urdf (robot description, URDF)
Before this commit: robot robot, 15 links, 14 joints
Links:
- added link LowerBody_link, mass 9.0; collision box size=0.300 0.080 0.550; visual box size=0.300 0.080 0.550
Joints:
- added joint Upper_Lower_Body_joint: type revolute, parent UpperBody_link, child LowerBody_link, origin xyz=0 0 0.500 rpy=0 0 0, axis 1 0 0, limit lower=0 upper=0 effort=500000 velocity=1000

Commit message: added limits to lowerbody_joint

File: urdf/robot.urdf (robot description, URDF)
Before this commit: robot robot, 16 links, 15 joints
Links:
- link LowerBody_link: mass 9.0 -> 5.0
- link UpperBody_link: mass 9.0 -> 40.0
Joints:
- joint Upper_Lower_Body_joint: limit lower=0 upper=0 effort=500000 velocity=1000 -> lower=-0.5708 upper=3.1415 effort=500000 velocity=1000; origin xyz=0 0 0.500 rpy=0 0 0 -> xyz=0 0 0.490 rpy=0 0 0

Commit message: added Bed as sdf for controller interaction

File: urdf/robot.urdf (robot description, URDF)
Before this commit: robot robot, 16 links, 15 joints
Links:
- removed link Bed_center_link
Joints:
- removed joint column_outside_Bedcenter_joint
