Commit message: using xacro to allow for easier and correct mass adjustmant respecting inertial properties

File: urdf/robot.urdf.xacro (robot description, xacro)
@@ -1,4 +1,4 @@
 <?xml version="1.0"?>
-<robot name="robot">
+<robot name="robot" xmlns:xacro="http://www.ros.org/wiki/xacro">
   <material name="blue">
     <color rgba="0 0 0.8 1"/>
@@ -60,5 +60,5 @@
     <child link = "frame_link" />
   </joint>
-  <!--Base frame-->
+  <!-- Base frame -->
   <link name="frame_link">
     <visual>
@@ -76,7 +76,12 @@
     </collision>
     <inertial>
-      <mass value="100.0"/>
+      <xacro:property name="frame_link_mass" value="100.0"/>
+      <mass value="${frame_link_mass}"/>
       <origin xyz="0 0 0.040" />
-      <inertia ixx="3.524" iyy="16.264" izz="19.789" ixy="0" ixz="0" iyz="0"/>
+      <inertia
+        ixx="${frame_link_mass / 12.0 * (0.645*0.645 + 0.080*0.080)}"
+        iyy="${frame_link_mass / 12.0 * (1.395*1.395 + 0.080*0.080)}"
+        izz="${frame_link_mass / 12.0 * (1.395*1.395 + 0.645*0.645)}"
+        ixy="0" ixz="0" iyz="0"/>
     </inertial>
   </link>
@@ -86,5 +91,5 @@
     <child link = "lower_motor_box_link" />
   </joint>
-  <!--lower motor box-->
+  <!-- lower motor box -->
   <link name="lower_motor_box_link">
     <visual>
@@ -102,7 +107,12 @@
     </collision>
     <inertial>
-      <mass value="28.0"/>
+      <xacro:property name="lower_motor_box_mass" value="28.0"/>
+      <mass value="${lower_motor_box_mass}"/>
       <origin xyz="0 0 0.110" />
-      <inertia ixx="0.196" iyy="0.194" izz="0.193" ixy="0" ixz="0" iyz="0"/>
+      <inertia
+        ixx="${lower_motor_box_mass / 12.0 * (0.218*0.218 + 0.220*0.220)}"
+        iyy="${lower_motor_box_mass / 12.0 * (0.2165*0.2165 + 0.220*0.220)}"
+        izz="${lower_motor_box_mass / 12.0 * (0.2165*0.2165 + 0.218*0.218)}"
+        ixy="0" ixz="0" iyz="0"/>
     </inertial>
   </link>
@@ -112,5 +122,5 @@
     <child link = "column_outside_link" />
   </joint>
-    <!--lifting_column_outside-->
+  <!-- lifting_column_outside -->
   <link name="column_outside_link">
     <visual>
@@ -128,7 +138,12 @@
     </collision>
     <inertial>
-      <mass value="0.5"/>
+      <xacro:property name="column_outside_mass" value="0.5"/>
+      <mass value="${column_outside_mass}"/>
       <origin xyz="0.065 0 0.320"/>
-      <inertia ixx="0.313" iyy="0.307" izz="0.031" ixy="0" ixz="0" iyz="0"/>
+      <inertia
+        ixx="${column_outside_mass / 12.0 * (0.202*0.202 + 0.640*0.640)}"
+        iyy="${column_outside_mass / 12.0 * (0.010*0.010 + 0.640*0.640)}"
+        izz="${column_outside_mass / 12.0 * (0.010*0.010 + 0.202*0.202)}"
+        ixy="0" ixz="0" iyz="0"/>
     </inertial>
   </link>
@@ -139,7 +154,7 @@
     <axis xyz="0 0 1" />
     <dynamics damping="0.5" friction="1.1"/>
-    <limit lower="0" upper="50.0" velocity="100" effort="5000"/> <!--only a lower limit and a realistically unachievable upper limit-->
-  </joint>
-  <!--lifting_column_inside-->
+    <limit lower="0" upper="50.0" velocity="100" effort="5000"/>
+  </joint>
+  <!-- lifting_column_inside -->
   <link name="column_inside_link">
     <visual>
@@ -157,7 +172,12 @@
     </collision>
     <inertial>
-      <mass value="9.0"/>
+      <xacro:property name="column_inside_mass" value="9.0"/>
+      <mass value="${column_inside_mass}"/>
       <origin xyz="0 0 0.320"/>
-      <inertia ixx="0.317" iyy="0.308" izz="0.047" ixy="0" ixz="0" iyz="0"/>
+      <inertia
+        ixx="${column_inside_mass / 12.0 * (0.177*0.177 + 0.640*0.640)}"
+        iyy="${column_inside_mass / 12.0 * (0.120*0.120 + 0.640*0.640)}"
+        izz="${column_inside_mass / 12.0 * (0.120*0.120 + 0.177*0.177)}"
+        ixy="0" ixz="0" iyz="0"/>
     </inertial>
   </link>
@@ -167,5 +187,5 @@
     <child link = "middle_motor_box_link" />
   </joint>
-  <!--middle motor box-->
+  <!-- middle motor box  -->
   <link name="middle_motor_box_link">
     <visual>
@@ -183,7 +203,12 @@
     </collision>
     <inertial>
-      <mass value="19.0"/>
+      <xacro:property name="middle_motor_box_mass" value="19.0"/>
+      <mass value="${middle_motor_box_mass}"/>
       <origin xyz="0 0 0.085"/>
-      <inertia ixx="0.092" iyy="0.092" izz="0.150" ixy="0" ixz="0" iyz="0"/>
+      <inertia
+        ixx="${middle_motor_box_mass / 12.0 * (0.218*0.218 + 0.170*0.170)}"
+        iyy="${middle_motor_box_mass / 12.0 * (0.218*0.218 + 0.170*0.170)}"
+        izz="${middle_motor_box_mass / 12.0 * (0.218*0.218 + 0.218*0.218)}"
+        ixy="0" ixz="0" iyz="0"/>
     </inertial>
   </link>
@@ -193,5 +218,5 @@
     <child link = "upper_cylinder_link" />
   </joint>
-  <!--cylinder connecting the upper boxes-->
+  <!-- cylinder connecting upper boxes -->
   <link name="upper_cylinder_link">
     <visual>
@@ -209,10 +234,15 @@
     </collision>
     <inertial>
-      <mass value="1.0"/>
+      <xacro:property name="upper_cylinder_mass" value="1.0"/>
+      <mass value="${upper_cylinder_mass}"/>
       <origin xyz="0 0 0.020"/>
-      <inertia ixx="0.007" iyy="0.007" izz="0.006" ixy="0" ixz="0" iyz="0"/>
-    </inertial>
-  </link>
-  <joint name = "upper_cylinder_upper_motor_joint" type = "continuous"> <!--coninuous = revolute with no limits -->
+      <inertia
+        ixx="${upper_cylinder_mass / 12.0 * (3*0.110*0.110 + 0.040*0.040)}"
+        iyy="${upper_cylinder_mass / 12.0 * (3*0.110*0.110 + 0.040*0.040)}"
+        izz="${upper_cylinder_mass / 2.0 * (0.110*0.110)}"
+        ixy="0" ixz="0" iyz="0"/>
+    </inertial>
+  </link>
+  <joint name = "upper_cylinder_upper_motor_joint" type = "continuous">
     <origin xyz="0 0 0.040"/>
     <parent link = "upper_cylinder_link" />
@@ -220,7 +250,6 @@
     <dynamics damping="0.5" friction="0.1"/>
     <axis xyz="0 0 1" />
-    <!-- <limit lower="-3.141" upper="1.5708" velocity="1000" effort="500000"/> -->
-  </joint>
-  <!--upper motor box-->
+  </joint>
+  <!-- upper motor box -->
   <link name="upper_motor_box_link">
     <visual>
@@ -238,10 +267,15 @@
     </collision>
     <inertial>
-      <mass value="22.0"/>
+      <xacro:property name="upper_motor_box_mass" value="22.0"/>
+      <mass value="${upper_motor_box_mass}"/>
       <origin xyz="-0.11575 0 0.08475"/>
-      <inertia ixx="0.161" iyy="0.677" izz="0.784" ixy="0" ixz="0" iyz="0"/>
-    </inertial>
-  </link>
-  <joint name="upper_motor_box_arm_joint" type="continuous"> <!--coninuous = revolute with no limits -->
+      <inertia
+        ixx="${upper_motor_box_mass / 12.0 * (0.223*0.223 + 0.1695*0.1695)}"
+        iyy="${upper_motor_box_mass / 12.0 * (0.4215*0.4215 + 0.1695*0.1695)}"
+        izz="${upper_motor_box_mass / 12.0 * (0.4215*0.4215 + 0.223*0.223)}"
+        ixy="0" ixz="0" iyz="0"/>
+    </inertial>
+  </link>
+  <joint name="upper_motor_box_arm_joint" type="continuous">
     <parent link="upper_motor_box_link"/>
     <child link="arm_first_link"/>
@@ -249,7 +283,6 @@
     <dynamics damping="0.5" friction="0.1"/>
     <axis xyz="0 0 1" rpy="0 0 0"/>
-    <!-- <limit lower="-1.5708" upper="0" velocity="1000" effort="5000"/>-->
-  </joint>
-  <!--first arm link-->
+  </joint>
+  <!-- arm_first_link -->
   <link name="arm_first_link">
     <visual>
@@ -267,7 +300,12 @@
     </collision>
     <inertial>
-      <mass value="1.5"/>
+      <xacro:property name="arm_first_mass" value="1.5"/>
+      <mass value="${arm_first_mass}"/>
       <origin xyz="0 0 0.074" rpy="0 0 0" />
-      <inertia ixx="0.003" iyy="0.003" izz="0.0001688" ixy="0" ixz="0" iyz="0"/>
+      <inertia
+        ixx="${arm_first_mass / 12.0 * (3*0.015*0.015 + 0.148*0.148)}"
+        iyy="${arm_first_mass / 12.0 * (3*0.015*0.015 + 0.148*0.148)}"
+        izz="${arm_first_mass / 2.0 * (0.015*0.015)}"
+        ixy="0" ixz="0" iyz="0"/>
     </inertial>
   </link>
@@ -277,4 +315,5 @@
     <origin xyz="0 0 0.148" rpy="0 -1.5708 0"/>
   </joint>
+  <!-- arm_second_link -->
   <link name="arm_second_link">
     <visual>
@@ -292,7 +331,12 @@
     </collision>
     <inertial>
-      <mass value="0.5"/>
+      <xacro:property name="arm_second_mass" value="0.5"/>
+      <mass value="${arm_second_mass}"/>
       <origin xyz="0 0 0.153" rpy="0 0 0"/>
-      <inertia ixx="0.004" iyy="0.004" izz="0.0000563" ixy="0" ixz="0" iyz="0"/>
+      <inertia
+        ixx="${arm_second_mass / 12.0 * (3*0.015*0.015 + 0.306*0.306)}"
+        iyy="${arm_second_mass / 12.0 * (3*0.015*0.015 + 0.306*0.306)}"
+        izz="${arm_second_mass / 2.0 * (0.015*0.015)}"
+        ixy="0" ixz="0" iyz="0"/>
     </inertial>
   </link>
@@ -302,4 +346,5 @@
     <origin xyz="0 0 0.314" rpy="0 1.5708 0"/>
   </joint>
+  <!-- arm_third_link -->
   <link name="arm_third_link">
     <visual>
@@ -317,7 +362,12 @@
     </collision>
     <inertial>
-      <mass value="2.5"/>
+      <xacro:property name="arm_third_mass" value="2.5"/>
+      <mass value="${arm_third_mass}"/>
       <origin xyz="0 0 0.419"/>
-      <inertia ixx="0.146" iyy="0.146" izz="0.0002813" ixy="0" ixz="0" iyz="0"/>
+      <inertia
+        ixx="${arm_third_mass / 12.0 * (3*0.015*0.015 + 0.838*0.838)}"
+        iyy="${arm_third_mass / 12.0 * (3*0.015*0.015 + 0.838*0.838)}"
+        izz="${arm_third_mass / 2.0 * (0.015*0.015)}"
+        ixy="0" ixz="0" iyz="0"/>
     </inertial>
   </link>
@@ -329,5 +379,5 @@
     <axis xyz="1 0 0" />
   </joint>
-  <!--BodyArms-->
+  <!-- BodyArms -->
   <link name="BodyArms_link">
     <visual>
@@ -345,7 +395,12 @@
     </collision>
     <inertial>
-      <mass value="9.0"/>
+      <xacro:property name="body_arms_mass" value="9.0"/>
+      <mass value="${body_arms_mass}"/>
       <origin xyz="0 0.100 0.005"/>
-      <inertia ixx="0.317" iyy="0.308" izz="0.047" ixy="0" ixz="0" iyz="0"/>
+      <inertia
+        ixx="${body_arms_mass / 12.0 * (0.200*0.200 + 0.040*0.040)}"
+        iyy="${body_arms_mass / 12.0 * (0.400*0.400 + 0.040*0.040)}"
+        izz="${body_arms_mass / 12.0 * (0.400*0.400 + 0.200*0.200)}"
+        ixy="0" ixz="0" iyz="0"/>
     </inertial>
   </link>
@@ -355,4 +410,5 @@
     <child link = "UpperBody_link" />
   </joint>
+  <!-- UpperBody -->
   <link name="UpperBody_link">
     <visual>
@@ -370,7 +426,12 @@
     </collision>
     <inertial>
-      <mass value="40.0"/>
+      <xacro:property name="upper_body_mass" value="20.0"/>
+      <mass value="${upper_body_mass}"/>
       <origin xyz="0 0 0.20"/>
-      <inertia ixx="0.317" iyy="0.308" izz="0.047" ixy="0" ixz="0" iyz="0"/>
+      <inertia
+        ixx="${upper_body_mass / 12.0 * (0.100*0.100 + 0.550*0.550)}"
+        iyy="${upper_body_mass / 12.0 * (0.400*0.400 + 0.550*0.550)}"
+        izz="${upper_body_mass / 12.0 * (0.400*0.400 + 0.100*0.100)}"
+        ixy="0" ixz="0" iyz="0"/>
     </inertial>
   </link>
@@ -383,4 +444,5 @@
     <limit lower="-0.5708" upper="3.1415" velocity="1000" effort="500000"/>
   </joint>
+  <!-- LowerBody -->
   <link name="LowerBody_link">
     <visual>
@@ -398,7 +460,12 @@
     </collision>
     <inertial>
-      <mass value="5.0"/>
+      <xacro:property name="lower_body_mass" value="5.0"/>
+      <mass value="${lower_body_mass}"/>
       <origin xyz="0 0 0.275"/>
-      <inertia ixx="0.317" iyy="0.308" izz="0.047" ixy="0" ixz="0" iyz="0"/>
+      <inertia
+        ixx="${lower_body_mass / 12.0 * (0.080*0.080 + 0.550*0.550)}"
+        iyy="${lower_body_mass / 12.0 * (0.300*0.300 + 0.550*0.550)}"
+        izz="${lower_body_mass / 12.0 * (0.300*0.300 + 0.080*0.080)}"
+        ixy="0" ixz="0" iyz="0"/>
     </inertial>
   </link>
@@ -410,5 +477,4 @@
   <link name="end_effector" />
   <!-- Gazebo material references -->
-  <!-- Grey links (frame, lower motor boxes) -->
   <gazebo reference="frame_link">
     <material>Gazebo/Grey</material>
@@ -423,10 +489,9 @@
     <material>Gazebo/Grey</material>
   </gazebo>
-  <!-- White links (columns, cylinder) -->
   <gazebo reference="column_outside_link">
     <material>Gazebo/White</material>
   </gazebo>
   <gazebo reference="BodyArms_link">
-  <material>Gazebo/White</material>
+    <material>Gazebo/White</material>
   </gazebo>
   <gazebo reference="UpperBody_link">
@@ -442,5 +507,4 @@
     <material>Gazebo/White</material>
   </gazebo>
-  <!-- Blue links (arm segments) -->
   <gazebo reference="arm_first_link">
     <material>Gazebo/Blue</material>

Commit message: added comments explaining the changes. expecially the urdf of the robot

File: urdf/robot.urdf.xacro (robot description, xacro)
@@ -1,2 +1,37 @@
+<!--
+  This is the URDF file for the robot model used in the Gazebo simulation. It defines the robot's structure, including its links, joints, and physical properties.
+  The robot consists of a base frame, a lifting column with two parts (inside and outside), three motor boxes (lower, middle, upper), an arm with three segments, and a body with upper and lower parts.
+  The collsion and inertial properties all match the visual properties of the links.
+  There is a simplyfied model of a patient attached to the robot arm to simulate the weight of a human body and its effect on the robot's movement.
+  To make the weight of the patient easily adjustable, the mass of the patient can be changed by modifying the mass values of the links.
+  This is also the main reason why the file is .xacro instead of .urdf, to allow for the use of xacro properties to easily adjust the mass values of the links without having to manually recalculate the correct inertia values each time.
+  To make the inertia calculation easy for the developer the links are modeled as simple geometric shapes (boxes and cylinders) that are combined with fixed joints.(gazebo collapses links connected by fixed joints into a single link)
+  The robot has three joints that are controlled with ROS2 control:
+    the column_outside_column_inside_joint (prismatic joint for height),
+    the upper_cylinder_upper_motor_joint (continuous joint for rotation),
+    and the upper_motor_box_arm_joint (continuous joint for arm rotation).
+  The robot structure with all its links in short is as follows:
+  first link:
+  - robot_base
+  - frame_link
+  - lower_motor_box_link
+  - column_outside_link
+  second link:
+  - column_inside_link
+  - middle_motor_box_link
+  - upper_cylinder_link
+  third link:
+  - upper_motor_box_link
+  fourth link:
+  - arm_first_link
+  - arm_second_link
+  - arm_third_link
+  Patient link:(loosely attached to the arm with a continuous joint but without actuator) (providing actuators can be subject of a future work to simulate patient movement)
+  - BodyArms_link (link)
+  - UpperBody_link (link)
+  (looslely attached to the upper body with a revolute joint with limits but also without actuator) (providing actuators can be subject of a future work to simulate patient movement)
+  - LowerBody_link (link)
+  (- end_effector (link))
+-->
 <?xml version="1.0"?>
 <robot name="robot" xmlns:xacro="http://www.ros.org/wiki/xacro">
@@ -21,5 +56,5 @@
       <plugin>gazebo_ros2_control/GazeboSystem</plugin>
     </hardware>
-    <joint name="upper_cylinder_upper_motor_joint">
+    <joint name="upper_cylinder_upper_motor_joint"> <!-- rotation joint -->
       <command_interface name="effort"/>
       <state_interface name="position">
@@ -29,5 +64,5 @@
       <state_interface name="effort"/>
     </joint>
-    <joint name="column_outside_column_inside_joint">
+    <joint name="column_outside_column_inside_joint"> <!-- height joint -->
       <command_interface name="effort"/>
       <state_interface name="position">
@@ -37,5 +72,5 @@
       <state_interface name="effort"/>
     </joint>
-    <joint name="upper_motor_box_arm_joint">
+    <joint name="upper_motor_box_arm_joint">  <!-- arm rotation joint -->
       <command_interface name="effort"/>
       <state_interface name="position">
@@ -107,5 +142,5 @@
     </collision>
     <inertial>
-      <xacro:property name="lower_motor_box_mass" value="28.0"/>
+      <xacro:property name="lower_motor_box_mass" value="28.0"/> <!-- mass of the lower motor box AND the outside column (see mass property of outside column for explanation) -->
       <mass value="${lower_motor_box_mass}"/>
       <origin xyz="0 0 0.110" />
@@ -138,5 +173,5 @@
     </collision>
     <inertial>
-      <xacro:property name="column_outside_mass" value="0.5"/>
+      <xacro:property name="column_outside_mass" value="0.5"/> <!-- mass of the outside column is near zero because it is a simplification for the collsion and visual representation that is a bad inertial representation. The mass is added to the lower motor box instead.-->
       <mass value="${column_outside_mass}"/>
       <origin xyz="0.065 0 0.320"/>
@@ -476,5 +511,5 @@
   </joint>
   <link name="end_effector" />
-  <!-- Gazebo material references -->
+  <!-- Gazebo material references. only for color purposes -->
   <gazebo reference="frame_link">
     <material>Gazebo/Grey</material>

Commit message: cleaned up unused files that i created. made some last changes.

File: urdf/robot.urdf.xacro (robot description, xacro)
@@ -1,14 +1,13 @@
 <!--
-  This is the URDF file for the robot model used in the Gazebo simulation. It defines the robot's structure, including its links, joints, and physical properties.
-  The robot consists of a base frame, a lifting column with two parts (inside and outside), three motor boxes (lower, middle, upper), an arm with three segments, and a body with upper and lower parts.
+  This is the URDF file for the robot model used in the Gazebo simulation.
   The collsion and inertial properties all match the visual properties of the links.
-  There is a simplyfied model of a patient attached to the robot arm to simulate the weight of a human body and its effect on the robot's movement.
+  There is a simplified model of a patient attached to the robot arm to simulate the weight of a human body and its effect on the robot's movement.
   To make the weight of the patient easily adjustable, the mass of the patient can be changed by modifying the mass values of the links.
-  This is also the main reason why the file is .xacro instead of .urdf, to allow for the use of xacro properties to easily adjust the mass values of the links without having to manually recalculate the correct inertia values each time.
+  This is also the main reason why the file is .urdf.xacro instead of .urdf, to allow for the use of xacro properties to easily adjust the mass values of the links without having to manually recalculate the correct inertia values each time.
   To make the inertia calculation easy for the developer the links are modeled as simple geometric shapes (boxes and cylinders) that are combined with fixed joints.(gazebo collapses links connected by fixed joints into a single link)
   The robot has three joints that are controlled with ROS2 control:
-    the column_outside_column_inside_joint (prismatic joint for height),
-    the upper_cylinder_upper_motor_joint (continuous joint for rotation),
-    and the upper_motor_box_arm_joint (continuous joint for arm rotation).
+    column_outside_column_inside_joint (prismatic joint for height),
+    upper_cylinder_upper_motor_joint (continuous joint for rotation),
+    upper_motor_box_arm_joint (continuous joint for arm rotation).
   The robot structure with all its links in short is as follows:
   first link:
@@ -27,8 +26,8 @@
   - arm_second_link
   - arm_third_link
-  Patient link:(loosely attached to the arm with a continuous joint but without actuator) (providing actuators can be subject of a future work to simulate patient movement)
+  Patient link:(loosely attached to the arm with a continuous joint but without actuator) (providing actuators can be subject of a future work to simulate movement of the patient)
   - BodyArms_link (link)
   - UpperBody_link (link)
-  (looslely attached to the upper body with a revolute joint with limits but also without actuator) (providing actuators can be subject of a future work to simulate patient movement)
+  (looslely attached to the upper body with a revolute joint with limits but also without actuator) (providing actuators can be subject of a future work to simulate movement of the patient)
   - LowerBody_link (link)
   (- end_effector (link))
@@ -51,5 +50,5 @@
     <color rgba="0.84375 0.70703125 0.53515625 1"/>
   </material>
-  <!--define initial values-->
+  <!--define initial joint configurations-->
   <ros2_control name="GazeboSystem" type="system">
     <hardware>
@@ -111,5 +110,5 @@
     </collision>
     <inertial>
-      <xacro:property name="frame_link_mass" value="100.0"/>
+      <xacro:property name="frame_link_mass" value="200.0"/> <!-- especially high to stabilize-->
       <mass value="${frame_link_mass}"/>
       <origin xyz="0 0 0.040" />
@@ -461,5 +460,5 @@
     </collision>
     <inertial>
-      <xacro:property name="upper_body_mass" value="20.0"/>
+      <xacro:property name="upper_body_mass" value="40.0"/>
       <mass value="${upper_body_mass}"/>
       <origin xyz="0 0 0.20"/>
@@ -477,5 +476,5 @@
     <dynamics damping="0.5" friction="0.1"/>
     <axis xyz="1 0 0" />
-    <limit lower="-0.5708" upper="3.1415" velocity="1000" effort="500000"/>
+    <limit lower="-0.5708" upper="2.00" velocity="1000" effort="500000"/>
   </joint>
   <!-- LowerBody -->
@@ -495,5 +494,5 @@
     </collision>
     <inertial>
-      <xacro:property name="lower_body_mass" value="5.0"/>
+      <xacro:property name="lower_body_mass" value="30.0"/>
       <mass value="${lower_body_mass}"/>
       <origin xyz="0 0 0.275"/>
