Commit message: feat: aan_control.py - Helloise Trajektorie richtig abgespielt; fix: URDF Beine ohne Kollision; fix: launch FIle startet trajectory control (kein Argument mehr beim launchen)

File: urdf/robot.urdf.xacro (robot description, xacro)
@@ -21,28 +21,34 @@
       <plugin>gazebo_ros2_control/GazeboSystem</plugin>
     </hardware>
-    <joint name="upper_cylinder_upper_motor_joint"> <!-- rotation joint -->
-      <command_interface name="effort"/>
-      <state_interface name="position">
-        <param name="initial_value">0</param>
-      </state_interface>
-      <state_interface name="velocity"/>
-      <state_interface name="effort"/>
-    </joint>
-    <joint name="column_outside_column_inside_joint"> <!-- height joint -->
-      <command_interface name="effort"/>
-      <state_interface name="position">
-        <param name="initial_value">0.0</param>
-      </state_interface>
-      <state_interface name="velocity"/>
-      <state_interface name="effort"/>
-    </joint>
-    <joint name="upper_motor_box_arm_joint">  <!-- arm rotation joint -->
-      <command_interface name="effort"/>
-      <state_interface name="position">
-        <param name="initial_value">0</param>
-      </state_interface>
-      <state_interface name="velocity"/>
-      <state_interface name="effort"/>
-    </joint>
+      <joint name="upper_cylinder_upper_motor_joint"> <!-- rotation joint -->
+        <command_interface name="position"/>
+        <command_interface name="velocity"/>
+        <command_interface name="effort"/>
+        <state_interface name="position">
+          <param name="initial_value">0</param>
+        </state_interface>
+        <state_interface name="velocity"/>
+        <state_interface name="effort"/>
+      </joint>
+      <joint name="column_outside_column_inside_joint"> <!-- height joint -->
+        <command_interface name="position"/>
+        <command_interface name="velocity"/>
+        <command_interface name="effort"/>
+        <state_interface name="position">
+          <param name="initial_value">0</param>
+        </state_interface>
+        <state_interface name="velocity"/>
+        <state_interface name="effort"/>
+      </joint>
+      <joint name="upper_motor_box_arm_joint">  <!-- arm rotation joint -->
+        <command_interface name="position"/>
+        <command_interface name="velocity"/>
+        <command_interface name="effort"/>
+        <state_interface name="position">
+          <param name="initial_value">0</param>
+        </state_interface>
+        <state_interface name="velocity"/>
+        <state_interface name="effort"/>
+      </joint>
   </ros2_control>
   <gazebo>
@@ -54,5 +60,5 @@
   </gazebo>
   <!-- The Robot Description starts here:-->
-  <link name="robot_base" />
+  <link name="robot_base"/>
   <joint name = "map_frame_joint" type = "fixed">
     <origin xyz="0.35575 -0.180 0"/>
@@ -76,5 +82,5 @@
     </collision>
     <inertial>
-      <xacro:property name="frame_link_mass" value="200.0"/> <!-- especially high to stabilize-->
+      <xacro:property name="frame_link_mass" value="20000.0"/> <!-- specially high to stabilize-->
       <mass value="${frame_link_mass}"/>
       <origin xyz="0 0 0.040" />
@@ -449,12 +455,12 @@
       <origin xyz="0 0 0.275"/>
       <geometry>
-        <box size="0.300 0.080 0.550"/>
+        <box size="0.300 0.080 0.90"/>
       </geometry>
       <material name="white"/>
     </visual>
     <collision>
-      <origin xyz="0 0 0.275"/>
-      <geometry>
-        <box size="0.300 0.080 0.550"/>
+      <origin xyz="0 0 0"/>
+      <geometry>
+        <box size="0 0 0"/>
       </geometry>
     </collision>

Commit message: feat: aan_control_minimal --> basic script that calculates the actuation torques using exemplary values

File: urdf/robot.urdf.xacro (robot description, xacro)
@@ -160,5 +160,5 @@
     <axis xyz="0 0 1" />
     <dynamics damping="0.5" friction="1.1"/>
-    <limit lower="0" upper="50.0" velocity="100" effort="5000"/>
+    <limit lower="0" upper="50.0" velocity="100" effort="500000"/>
   </joint>
   <!-- lifting_column_inside -->

Commit message: feat: effort controller integration

File: urdf/robot.urdf.xacro (robot description, xacro)
@@ -160,5 +160,5 @@
     <axis xyz="0 0 1" />
     <dynamics damping="0.5" friction="1.1"/>
-    <limit lower="0" upper="50.0" velocity="100" effort="500000"/>
+    <limit lower="0" upper="50.0" velocity="100" effort="5000"/>
   </joint>
   <!-- lifting_column_inside -->
@@ -432,5 +432,5 @@
     </collision>
     <inertial>
-      <xacro:property name="upper_body_mass" value="40.0"/>
+      <xacro:property name="upper_body_mass" value="50.0"/>
       <mass value="${upper_body_mass}"/>
       <origin xyz="0 0 0.20"/>
@@ -455,5 +455,5 @@
       <origin xyz="0 0 0.275"/>
       <geometry>
-        <box size="0.300 0.080 0.90"/>
+        <box size="0.300 0.080 0.30"/>
       </geometry>
       <material name="white"/>
@@ -462,9 +462,9 @@
       <origin xyz="0 0 0"/>
       <geometry>
-        <box size="0 0 0"/>
-      </geometry>
-    </collision>
-    <inertial>
-      <xacro:property name="lower_body_mass" value="30.0"/>
+        <box size="0.300 0.080 0.30"/>
+      </geometry>
+    </collision>
+    <inertial>
+      <xacro:property name="lower_body_mass" value="0.0"/>
       <mass value="${lower_body_mass}"/>
       <origin xyz="0 0 0.275"/>
